Commit message: Add files via upload

File: panda.urdf (robot description, URDF)
Before this commit: robot panda, 13 links, 12 joints
Links:
- removed link panda_hand
- removed link world
- added link base_link
- added link finger_tip, mass 0.73; collision mesh filename=package://franka_panda_description/meshes/collision/hand.stl; visual mesh filename=package://franka_panda_description/meshes/visual/hand.dae
Joints:
- joint panda_finger_joint1: parent panda_hand -> finger_tip
- joint panda_finger_joint2: parent panda_hand -> finger_tip
- joint panda_hand_joint: child panda_hand -> finger_tip
- joint panda_joint_world: parent world -> base_link
